File: hardware/gemini_right/gemini_right.kicad_pcb (KiCad board)
At the start: 2 copper layers, 0 parts

Commit message: initial routing for gemini_right
Parts:
- added C1: 2.2uF, Capacitor_SMD:C_0603_1608Metric_Pad1.08x0.95mm_HandSolder, F.Cu at (74.9, 107.1)
- added C10: 1uF, Capacitor_SMD:C_0603_1608Metric_Pad1.08x0.95mm_HandSolder, F.Cu at (67.7, 62.0)
- added C11: 22uF, Capacitor_SMD:C_0603_1608Metric_Pad1.08x0.95mm_HandSolder, F.Cu at (67.7, 58.3)
- added C12: 10uF, Capacitor_SMD:C_0603_1608Metric_Pad1.08x0.95mm_HandSolder, F.Cu at (162.4, 48.9)
- added C13: 10uF, Capacitor_SMD:C_0603_1608Metric_Pad1.08x0.95mm_HandSolder, F.Cu at (97.4, 118.7)
- added C14: 100nF, Capacitor_SMD:C_0603_1608Metric_Pad1.08x0.95mm_HandSolder, F.Cu at (103.5, 114.4)
- added C15: 100nF, Capacitor_SMD:C_0603_1608Metric_Pad1.08x0.95mm_HandSolder, F.Cu at (109.1, 114.4)
- added C16: 2.2uF, Capacitor_SMD:C_0603_1608Metric_Pad1.08x0.95mm_HandSolder, F.Cu at (72.2, 93.5)
- added C2: 10uF, Capacitor_SMD:C_0603_1608Metric_Pad1.08x0.95mm_HandSolder, F.Cu at (71.6, 83.4)
- added C3: 10uF, Capacitor_SMD:C_0603_1608Metric_Pad1.08x0.95mm_HandSolder, F.Cu at (72.4, 69.0)
- added C4: 22uF, Capacitor_SMD:C_0603_1608Metric_Pad1.08x0.95mm_HandSolder, F.Cu at (67.1, 89.9)
- added C5: 22uF, Capacitor_SMD:C_0603_1608Metric_Pad1.08x0.95mm_HandSolder, F.Cu at (67.1, 88.1)
- added C6: 22uF, Capacitor_SMD:C_0603_1608Metric_Pad1.08x0.95mm_HandSolder, F.Cu at (67.1, 86.3)
- added C7: 1uF, Capacitor_SMD:C_0603_1608Metric_Pad1.08x0.95mm_HandSolder, F.Cu at (70.6, 85.9)
- added C8: 1uF, Capacitor_SMD:C_0603_1608Metric_Pad1.08x0.95mm_HandSolder, F.Cu at (72.2, 91.7)
- added C9: 1uF, Capacitor_SMD:C_0603_1608Metric_Pad1.08x0.95mm_HandSolder, F.Cu at (70.5, 65.1)
- added D1: 1N4007, Diode_SMD:D_SOD-123F, F.Cu at (157.9, 64.2)
- added D10: 1N4007, Diode_SMD:D_SOD-123F, F.Cu at (100.8, 53.8)
- added D11: 1N4007, Diode_SMD:D_SOD-123F, F.Cu at (100.8, 72.9)
- added D12: 1N4007, Diode_SMD:D_SOD-123F, F.Cu at (100.8, 92.0)
- added D13: 1N4007, Diode_SMD:D_SOD-123F, F.Cu at (81.8, 56.5)
- added D14: 1N4007, Diode_SMD:D_SOD-123F, F.Cu at (81.8, 75.6)
- added D15: 1N4007, Diode_SMD:D_SOD-123F, F.Cu at (81.8, 94.8)
- added D16: 1N4007, Diode_SMD:D_SOD-123F, F.Cu at (108.3, 109.8)
- added D17: 1N4007, Diode_SMD:D_SOD-123F, F.Cu at (89.4, 113.1)
- added D18: 1N4007, Diode_SMD:D_SOD-123F, F.Cu at (75.1, 126.4)
- added D19: LED_WHITE, Diode_SMD:D_0603_1608Metric_Pad1.05x0.95mm_HandSolder, F.Cu at (159.2, 117.1)
- added D2: 1N4007, Diode_SMD:D_SOD-123F, F.Cu at (157.9, 83.4)
- added D20: LED_BLUE, Diode_SMD:D_0603_1608Metric_Pad1.05x0.95mm_HandSolder, F.Cu at (159.2, 115.2)
- added D3: 1N4007, Diode_SMD:D_SOD-123F, F.Cu at (157.9, 102.5)
- added D4: 1N4007, Diode_SMD:D_SOD-123F, F.Cu at (138.9, 56.5)
- added D5: 1N4007, Diode_SMD:D_SOD-123F, F.Cu at (138.9, 75.6)
- added D6: 1N4007, Diode_SMD:D_SOD-123F, F.Cu at (138.9, 94.8)
- added D7: 1N4007, Diode_SMD:D_SOD-123F, F.Cu at (119.8, 51.2)
- added D8: 1N4007, Diode_SMD:D_SOD-123F, F.Cu at (119.8, 70.4)
- added D9: 1N4007, Diode_SMD:D_SOD-123F, F.Cu at (119.8, 89.5)
- added IC1: XL9555__TSSOP-24_, SOP65P640X120-24N:SOP65P640X120-24N, F.Cu at (148.0, 112.3)
- added IC2: ESP32-C3-WROOM-02-N4, ESP32C3WROOM02N4:ESP32C3WROOM02N4, F.Cu at (129.8, 110.4)
- added J1: Conn_01x02_MountingPin, mx1.25_1x02_p1.25:CONN-SMD_2P-P1.25_XUNPU_WAFER-MX1.25-2PWB, F.Cu at (68.3, 52.8)
- added J1_toLeft1: USB_C_Receptacle_USB2.0_16P, Connector_USB:USB_C_Receptacle_GCT_USB4105-xx-A_16P_TopMnt_Horizontal, F.Cu at (67.6, 105.8)
- added J2: Conn_01x06_MountingPin, FPC_1x06_p0.5:FPC-SMD_6P-P0.50_XUNPU_FPC-05F-6PH20, F.Cu at (68.4, 95.1)
- added J2_toHost1: USB_C_Receptacle_USB2.0_16P, Connector_USB:USB_C_Receptacle_GCT_USB4105-xx-A_16P_TopMnt_Horizontal, F.Cu at (158.9, 41.7)
- added J3_passthrough1: USB_C_Receptacle_USB2.0_16P, Connector_USB:USB_C_Receptacle_GCT_USB4105-xx-A_16P_TopMnt_Horizontal, F.Cu at (94.4, 125.8)
- added L1: 1uH, Inductor_SMD:L_Sunlord_MWSA0402S, F.Cu at (68.2, 69.8)
- added R1: 470R, Resistor_SMD:R_0603_1608Metric_Pad0.98x0.95mm_HandSolder, F.Cu at (155.6, 117.1)
- added R10: 5.1kR, Resistor_SMD:R_0603_1608Metric_Pad0.98x0.95mm_HandSolder, F.Cu at (160.4, 48.9)
- added R11: 5.1kR, Resistor_SMD:R_0603_1608Metric_Pad0.98x0.95mm_HandSolder, F.Cu at (155.0, 48.9)
- added R12: 56kR, Resistor_SMD:R_0603_1608Metric_Pad0.98x0.95mm_HandSolder, F.Cu at (92.9, 118.7)
- added R13: 56kR, Resistor_SMD:R_0603_1608Metric_Pad0.98x0.95mm_HandSolder, F.Cu at (95.1, 118.7)
- added R14: 4.7kR, Resistor_SMD:R_0603_1608Metric_Pad0.98x0.95mm_HandSolder, F.Cu at (114.7, 114.4)
- added R2: 2kR, Resistor_SMD:R_0603_1608Metric_Pad0.98x0.95mm_HandSolder, F.Cu at (74.6, 102.1)
- added R3: 2kR, Resistor_SMD:R_0603_1608Metric_Pad0.98x0.95mm_HandSolder, F.Cu at (76.6, 102.1)
- added R4: 470R, Resistor_SMD:R_0603_1608Metric_Pad0.98x0.95mm_HandSolder, F.Cu at (155.6, 115.2)
- added R5: 2R, Resistor_SMD:R_0603_1608Metric_Pad0.98x0.95mm_HandSolder, F.Cu at (69.8, 82.0)
- added R6: 4.7kR, Resistor_SMD:R_0603_1608Metric_Pad0.98x0.95mm_HandSolder, F.Cu at (68.5, 65.1)
- added R7: 100R, Resistor_SMD:R_0603_1608Metric_Pad0.98x0.95mm_HandSolder, F.Cu at (72.4, 65.1)
- added R8: 470R, Resistor_SMD:R_0603_1608Metric_Pad0.98x0.95mm_HandSolder, F.Cu at (67.7, 60.1)
- added R9: 51kR, Resistor_SMD:R_0603_1608Metric_Pad0.98x0.95mm_HandSolder, F.Cu at (159.2, 113.4)
- added SW1: SW_Push, choc_v1v2_compatible_withLED:SW_Kailh_Choc_V1V2_1.00u, F.Cu at (157.8, 59.2)
- added SW10: SW_Push, choc_v1v2_compatible_withLED:SW_Kailh_Choc_V1V2_1.00u, F.Cu at (100.8, 48.8)
- added SW11: SW_Push, choc_v1v2_compatible_withLED:SW_Kailh_Choc_V1V2_1.00u, F.Cu at (100.8, 67.9)
- added SW12: SW_Push, choc_v1v2_compatible_withLED:SW_Kailh_Choc_V1V2_1.00u, F.Cu at (100.8, 87.0)
- added SW13: SW_Push, choc_v1v2_compatible_withLED:SW_Kailh_Choc_V1V2_1.00u, F.Cu at (81.8, 51.5)
- added SW14: SW_Push, choc_v1v2_compatible_withLED:SW_Kailh_Choc_V1V2_1.00u, F.Cu at (81.8, 70.6)
- added SW15: SW_Push, choc_v1v2_compatible_withLED:SW_Kailh_Choc_V1V2_1.00u, F.Cu at (81.8, 89.8)
- added SW16: SW_Push, choc_v1v2_compatible_withLED:SW_Kailh_Choc_V1V2_1.00u, F.Cu at (108.3, 104.8)
- added SW17: SW_Push, choc_v1v2_compatible_withLED:SW_Kailh_Choc_V1V2_1.00u, F.Cu at (88.1, 108.3)
- added SW18: SW_Push, choc_v1v2_compatible_withLED:SW_Kailh_Choc_V1V2_1.00u, F.Cu at (72.6, 122.0)
- added SW19: SW_Push, Button_Switch_SMD:SW_SPST_SKQG_WithoutStem, F.Cu at (159.3, 109.4)
- added SW2: SW_Push, choc_v1v2_compatible_withLED:SW_Kailh_Choc_V1V2_1.00u, F.Cu at (157.8, 78.4)
- added SW3: SW_Push, choc_v1v2_compatible_withLED:SW_Kailh_Choc_V1V2_1.00u, F.Cu at (157.8, 97.5)
- added SW4: SW_Push, choc_v1v2_compatible_withLED:SW_Kailh_Choc_V1V2_1.00u, F.Cu at (138.8, 51.5)
- added SW5: SW_Push, choc_v1v2_compatible_withLED:SW_Kailh_Choc_V1V2_1.00u, F.Cu at (138.8, 70.6)
- added SW6: SW_Push, choc_v1v2_compatible_withLED:SW_Kailh_Choc_V1V2_1.00u, F.Cu at (138.8, 89.8)
- added SW7: SW_Push, choc_v1v2_compatible_withLED:SW_Kailh_Choc_V1V2_1.00u, F.Cu at (119.8, 46.2)
- added SW8: SW_Push, choc_v1v2_compatible_withLED:SW_Kailh_Choc_V1V2_1.00u, F.Cu at (119.8, 65.4)
- added SW9: SW_Push, choc_v1v2_compatible_withLED:SW_Kailh_Choc_V1V2_1.00u, F.Cu at (119.8, 84.5)
- added U1: IP5407, IP5306_4.35V:SOIC127P600X165-9N, F.Cu at (69.4, 76.5)
- added U2: XC6206PxxxMR, Package_TO_SOT_SMD:SOT-23-3, F.Cu at (70.7, 88.8)
- added U3: CH9329, sop-16_L9.9-W3.9-P1.27-LS6.0:SOP-16_L9.9-W3.9-P1.27-LS6.0-BL, F.Cu at (107.3, 121.0)
- added U4: SL2.1s, ssop-16_L4.6-W2.6-P0.53-LS4.0:SSOP-16_L4.6-W2.6-P0.53-LS4.0-BL, F.Cu at (150.9, 47.9)
- added U5: CW2015CHBD, Package_DFN_QFN:TDFN-8-1EP_3x2mm_P0.5mm_EP1.4x1.4mm, F.Cu at (71.5, 61.1)
- added Y1: Crystal_GND24, Oscillator:Oscillator_SMD_Abracon_ASE-4Pin_3.2x2.5mm_HandSoldering, F.Cu at (150.9, 42.6)
Routing:
- net /VBUS: track 0.00 -> 202.4 mm, vias 0 -> 5
- net /RCOL0: track 0.00 -> 192.6 mm, vias 0 -> 1
- net /RCOL1: track 0.00 -> 174.1 mm, vias 0 -> 3
- net /PWR_BTN: track 0.00 -> 159.7 mm, vias 0 -> 2
- net /RCOL2: track 0.00 -> 149.2 mm, vias 0 -> 6
- net +3V3: track 0.00 -> 144.8 mm, vias 0 -> 4
- net /SDA: track 0.00 -> 136.2 mm, vias 0 -> 4
- net /SCL: track 0.00 -> 133.6 mm, vias 0 -> 4
- net /RROW4: track 0.00 -> 119.4 mm, vias 0 -> 4
- net /USB_PASSTHROUGH_DN: track 0.00 -> 117.2 mm, vias 0 -> 2
- net Net-(U1-LED1): track 0.00 -> 115.5 mm, vias 0 -> 2
- net /USB_PASSTHROUGH_DP: track 0.00 -> 113.7 mm, vias 0 -> 2
- net /PWR_STAT: track 0.00 -> 109.0 mm, vias 0 -> 2
- net /RROW3: track 0.00 -> 101.3 mm, vias 0 -> 4
- net /USB_HID_DN: track 0.00 -> 96.1 mm
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- added copper zone on F.Cu, net +3V3
- added copper zone on F.Cu, net +BATT
- added copper zone on F.Cu, net /5VOUT
- added copper zone on F.Cu, net /VBUS
- added copper zone on B.Cu, net GND
- added copper zone on F.Cu, net GND
- added copper zone on F.Cu, net Net-(U1-SW)
Other:
- board outline added: 99.8 x 93.2 mm

Commit message: test production 1
Parts:
- moved J2_toHost1 0.05 mm to (158.9, 41.8)
Routing:
- net /USB_DP: track 15.9 -> 14.2 mm
- net +3V3: track 144.8 -> 143.3 mm
- net /PWR_BTN: track 159.7 -> 160.6 mm
- net GND: vias 32 -> 40
