File: hardware/gemini_right/gemini_right.kicad_pcb (KiCad board)
At the start: 2 copper layers, 99.8 x 93.2 mm, 80 parts, among them IC1 CW2015CHBD, IC2 XL9555__TSSOP-24_, J1 Conn_01x06_MountingPin, J1_toLeft1 USB_C_Receptacle_USB2.0_16P, J2 Conn_01x02_MountingPin, J2_toHost1 USB_C_Receptacle_USB2.0_16P, SW1 SW_Push, SW10 SW_Push, SW11 SW_Push, SW12 SW_Push, SW13 SW_Push, SW14 SW_Push, SW15 SW_Push, SW16 SW_Push, SW17 SW_Push, SW18 SW_Push, SW19 SW_Push, SW2 SW_Push, SW20 SW_Push, SW3 SW_Push, SW4 SW_Push, SW5 SW_Push, SW6 SW_Push, SW7 SW_Push, SW8 SW_Push, SW9 SW_Push, U1 ETA9742, U2 XC6206PxxxMR, U3 CH582F, Y1 32.768khz 12.5pF 20ppm, Y2 32Mhz 12pF 10ppm

Commit message: update capacitor
Parts:
- C14: value 0.1uF -> 2.2uF
- C15: value 1uF -> 2.2uF

Commit message: use esp32c3 instead
Parts:
- removed AE1: Antenna_Shield, chxxx_antenna:ANT-F-3-2.4G-1.6mmFR4-WCH_mirror
- removed C14, C15: 2.2uF, Capacitor_SMD:C_0603_1608Metric_Pad1.08x0.95mm_HandSolder
- removed L2: 10uH, Inductor_SMD:L_Chilisin_BMRA00040420
- removed SW20: SW_Push, Button_Switch_SMD:SW_Tactile_SPST_NO_Straight_CK_PTS636Sx25SMTRLFS
- removed Y1: 32.768khz 12.5pF 20ppm, Crystal:Crystal_SMD_3215-2Pin_3.2x1.5mm
- removed Y2: 32Mhz 12pF 10ppm, Crystal:Crystal_SMD_3225-4Pin_3.2x2.5mm
- added C5: 1uF, Capacitor_SMD:C_0603_1608Metric_Pad1.08x0.95mm_HandSolder, F.Cu at (144.4, 113.5)
- added R12: 4.7k, Resistor_SMD:R_0603_1608Metric_Pad0.98x0.95mm_HandSolder, F.Cu at (148.0, 113.5)
- added R13: 10k, Resistor_SMD:R_0603_1608Metric_Pad0.98x0.95mm_HandSolder, F.Cu at (141.5, 111.0)
- C12: value 0.1uF -> 100nF
- U3: value CH582F -> ESP32-C3-WROOM-02; footprint chxxx:QFN28_4X4 -> RF_Module:ESP32-C3-WROOM-02
- moved C8 22.7 mm to (144.4, 109.2), turned to 180 degrees
- moved C12 17.1 mm to (144.4, 111.8)
- moved SW19 11.4 mm to (153.5, 111.0)
- moved IC2 5.67 mm to (144.5, 101.8)
- moved R4 3.16 mm to (120.1, 98.0), turned to 180 degrees
- moved U3 3.15 mm to (128.1, 106.2), turned to 180 degrees
- turned D19 to 180 degrees
- turned D20 to 180 degrees
Connections:
- C12 pad 2: /VDCIA -> +3V3
- C8 pad 2: Net-(U3-VINTA) -> Net-(U3-EN)
- D19 pad 1: /STAT_LED -> Net-(D19-K)
- D19 pad 2: Net-(D19-A) -> /STAT_LED
- D20 pad 1: /WARN_LED -> Net-(D20-K)
- D20 pad 2: Net-(D20-A) -> /WARN_LED
- R10 pad 1: Net-(D20-A) -> Net-(D20-K)
- R10 pad 2: /VBUS -> GND
- R9 pad 1: Net-(D19-A) -> Net-(D19-K)
- R9 pad 2: /VBUS -> GND
- SW19 pad 1: /ISPn -> /BOOTn
- U3 pad 1: /X32k_PIN0 -> +3V3
- U3 pad 10: /SCL -> /PWR_ALRT
- U3 pad 11: /SDA -> /TPAD_RDY
- U3 pad 12: /USB_D+ -> /TPAD_NRST
- U3 pad 14: /TPAD_NRST -> /USB_D+
- U3 pad 16: /RSTn -> /PWR_STAT
- U3 pad 17: /ISPn -> /BOOST_STAT
- U3 pad 18: /X32M_PIN1 -> /BOOTn
- U3 pad 19: /X32M_PIN0 -> GND
- U3 pad 2: /X32k_PIN1 -> Net-(U3-EN)
- U3 pad 3: /VDCIA -> /WARN_LED
- U3 pad 4: /VSW -> /STAT_LED
- U3 pad 5: +3V3 -> unconnected-(U3-IO6-Pad5)
- U3 pad 6: unconnected-(U3-PA8/RXD1/AIN12-Pad6) -> /KEY_INT
- U3 pad 7: /KEY_INT -> /SCL
- U3 pad 8: /PWR_ALRT -> /SDA
- U3 pad 9: /TPAD_RDY -> GND
Routing:
- net /VBUS: track 187.1 -> 121.9 mm, vias 5 -> 2
- net /RSTn: track 37.2 -> 0.00 mm, vias 2 -> 0
- net /RROW3: track 86.2 -> 52.5 mm, vias 7 -> 2
- net /BOOTn: track 0.00 -> 32.5 mm, vias 0 -> 2
- net +3V3: track 140.2 -> 160.8 mm
- net /ISPn: track 18.9 -> 0.00 mm, vias 2 -> 0
- net /USB_D-: track 78.9 -> 97.4 mm
- net /USB_D+: track 78.6 -> 96.8 mm
- net /RROW1: track 47.4 -> 32.6 mm, vias 2 -> 0
- net /SCL: track 156.1 -> 143.9 mm, vias 8 -> 6
- net /WARN_LED: track 32.9 -> 21.7 mm
- net /STAT_LED: track 32.3 -> 21.3 mm
- net /KEY_INT: track 87.0 -> 97.1 mm, vias 3 -> 2
- net /SDA: track 158.7 -> 149.6 mm, vias 8 -> 6
- net /VDCIA: track 8.94 -> 0.00 mm, vias 2 -> 0
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- added copper zone on F.Cu, net /BOOTn
- removed copper zone on F.Cu, net /ISPn
- removed copper zone on F.Cu, net /RSTn
- removed copper zone on F.Cu, net /VDCIA
Other:
- outline, holes or cut-outs redrawn
